File: DevBoard_NCP1090_KiCAD/DevBoard_NCP1090.sch (KiCad schematic (older format))
At the start: 12 parts, among them U1 NCP1090, X1 Conn_01x04, X2 Conn_01x03

Commit message: v2 initial commit
Parts:
- removed TP1, TP2: MountingHole_Pad, Measurement_Points:Measurement_Point_Round-SMD-Pad_Small, symbol Mechanical:MountingHole_Pad
Changed lines of the file:
@@
 Sheet 1 1
 Title "NCP1090 Development Board"
-Date "2018-08-19"
-Rev "1"
+Date "2018-09-08"
+Rev "2"
 Comp "Alex M."
 Comment1 ""
@@
 BR2b
 $Comp
-L Mechanical:MountingHole_Pad TP2
-U 1 1 5B7A2B37
-P 4300 4400
-F 0 "TP2" H 4200 4404 50  0000 R CNN
-F 1 "MountingHole_Pad" H 4400 4360 50  0001 L CNN
-F 2 "Measurement_Points:Measurement_Point_Round-SMD-Pad_Small" H 4300 4400 50  0001 C CNN
-F 3 "~" H 4300 4400 50  0001 C CNN
-	1    4300 4400
-	-1   0    0    1
-$EndComp
-$Comp
-L Mechanical:MountingHole_Pad TP1
-U 1 1 5B7A4029
-P 4300 2400
-F 0 "TP1" H 4400 2405 50  0000 L CNN
-F 1 "MountingHole_Pad" H 4400 2360 50  0001 L CNN
-F 2 "Measurement_Points:Measurement_Point_Round-SMD-Pad_Small" H 4300 2400 50  0001 C CNN
-F 3 "~" H 4300 2400 50  0001 C CNN
-	1    4300 2400
-	1    0    0    -1
-$EndComp
-$Comp
 L Connector_Generic:Conn_01x03 X2
